Commit message: ui updates, plus ability to run ros2 stuff and multiple processes

File: src/urdf/g1_29dof_with_hand.urdf (robot description, URDF)
Before this commit: robot g1_29dof_with_hand, 55 links, 54 joints
Links:
- link head_link: geometry collision mesh filename=meshes/head_link.stl; visual mesh filename=meshes/head_link.stl
- link left_ankle_pitch_link: geometry collision mesh filename=meshes/left_ankle_pitch_link.stl; visual mesh filename=meshes/left_ankle_pitch_link.stl
- link left_ankle_roll_link: geometry collision sphere radius=0.005; collision sphere radius=0.005
- link left_elbow_link: geometry collision mesh filename=meshes/left_elbow_link.stl; visual mesh filename=meshes/left_elbow_link.stl
- link left_hand_index_0_link: geometry collision mesh filename=meshes/left_hand_index_0_link.stl; visual mesh filename=meshes/left_hand_index_0_link.stl
- link left_hand_index_1_link: geometry collision mesh filename=meshes/left_hand_index_1_link.stl; visual mesh filename=meshes/left_hand_index_1_link.stl
- link left_hand_middle_0_link: geometry collision mesh filename=meshes/left_hand_middle_0_link.stl; visual mesh filename=meshes/left_hand_middle_0_link.stl
- link left_hand_middle_1_link: geometry collision mesh filename=meshes/left_hand_middle_1_link.stl; visual mesh filename=meshes/left_hand_middle_1_link.stl
- link left_hand_palm_link: geometry collision mesh filename=meshes/left_hand_palm_link.stl; visual mesh filename=meshes/left_hand_palm_link.stl
- link left_hand_thumb_0_link: geometry collision mesh filename=meshes/left_hand_thumb_0_link.stl; visual mesh filename=meshes/left_hand_thumb_0_link.stl
- link left_hand_thumb_1_link: geometry collision box size=0.02 0.03 0.02; visual mesh filename=meshes/left_hand_thumb_1_link.stl
- link left_hand_thumb_2_link: geometry collision mesh filename=meshes/left_hand_thumb_2_link.stl; visual mesh filename=meshes/left_hand_thumb_2_link.stl
- link left_hip_pitch_link: geometry collision mesh filename=meshes/left_hip_pitch_link.stl; visual mesh filename=meshes/left_hip_pitch_link.stl
- link left_hip_roll_link: geometry collision mesh filename=meshes/left_hip_roll_link.stl; visual mesh filename=meshes/left_hip_roll_link.stl
- link left_hip_yaw_link: geometry collision mesh filename=meshes/left_hip_yaw_link.stl; visual mesh filename=meshes/left_hip_yaw_link.stl
- link left_knee_link: geometry collision mesh filename=meshes/left_knee_link.stl; visual mesh filename=meshes/left_knee_link.stl
- link left_shoulder_pitch_link: geometry collision cylinder length=0.05 radius=0.03; visual mesh filename=meshes/left_shoulder_pitch_link.stl
- link left_shoulder_roll_link: geometry collision cylinder length=0.03 radius=0.03; visual mesh filename=meshes/left_shoulder_roll_link.stl
- link left_shoulder_yaw_link: geometry collision mesh filename=meshes/left_shoulder_yaw_link.stl; visual mesh filename=meshes/left_shoulder_yaw_link.stl
- link left_wrist_pitch_link: geometry collision mesh filename=meshes/left_wrist_pitch_link.stl; visual mesh filename=meshes/left_wrist_pitch_link.stl
- link left_wrist_roll_link: geometry collision mesh filename=meshes/left_wrist_roll_link.stl; visual mesh filename=meshes/left_wrist_roll_link.stl
- link left_wrist_yaw_link: geometry collision mesh filename=meshes/left_wrist_yaw_link.stl; visual mesh filename=meshes/left_wrist_yaw_link.stl
- link logo_link: geometry collision mesh filename=meshes/logo_link.stl; visual mesh filename=meshes/logo_link.stl
- link pelvis_contour_link: geometry collision mesh filename=meshes/pelvis_contour_link.stl; visual mesh filename=meshes/pelvis_contour_link.stl
- link right_ankle_pitch_link: geometry collision mesh filename=meshes/right_ankle_pitch_link.stl; visual mesh filename=meshes/right_ankle_pitch_link.stl
- link right_ankle_roll_link: geometry collision sphere radius=0.005; collision sphere radius=0.005
- link right_elbow_link: geometry collision mesh filename=meshes/right_elbow_link.stl; visual mesh filename=meshes/right_elbow_link.stl
- link right_hand_index_0_link: geometry collision mesh filename=meshes/right_hand_index_0_link.stl; visual mesh filename=meshes/right_hand_index_0_link.stl
- link right_hand_index_1_link: geometry collision mesh filename=meshes/right_hand_index_1_link.stl; visual mesh filename=meshes/right_hand_index_1_link.stl
- link right_hand_middle_0_link: geometry collision mesh filename=meshes/right_hand_middle_0_link.stl; visual mesh filename=meshes/right_hand_middle_0_link.stl
- link right_hand_middle_1_link: geometry collision mesh filename=meshes/right_hand_middle_1_link.stl; visual mesh filename=meshes/right_hand_middle_1_link.stl
- link right_hand_palm_link: geometry collision mesh filename=meshes/right_hand_palm_link.stl; visual mesh filename=meshes/right_hand_palm_link.stl
- link right_hand_thumb_0_link: geometry collision mesh filename=meshes/right_hand_thumb_0_link.stl; visual mesh filename=meshes/right_hand_thumb_0_link.stl
- link right_hand_thumb_1_link: geometry collision box size=0.02 0.03 0.02; visual mesh filename=meshes/right_hand_thumb_1_link.stl
- link right_hand_thumb_2_link: geometry collision mesh filename=meshes/right_hand_thumb_2_link.stl; visual mesh filename=meshes/right_hand_thumb_2_link.stl
- link right_hip_pitch_link: geometry collision mesh filename=meshes/right_hip_pitch_link.stl; visual mesh filename=meshes/right_hip_pitch_link.stl
- link right_hip_roll_link: geometry collision mesh filename=meshes/right_hip_roll_link.stl; visual mesh filename=meshes/right_hip_roll_link.stl
- link right_hip_yaw_link: geometry collision mesh filename=meshes/right_hip_yaw_link.stl; visual mesh filename=meshes/right_hip_yaw_link.stl
- link right_knee_link: geometry collision mesh filename=meshes/right_knee_link.stl; visual mesh filename=meshes/right_knee_link.stl
- link right_shoulder_pitch_link: geometry collision cylinder length=0.05 radius=0.03; visual mesh filename=meshes/right_shoulder_pitch_link.stl
- link right_shoulder_roll_link: geometry collision cylinder length=0.03 radius=0.03; visual mesh filename=meshes/right_shoulder_roll_link.stl
- link right_shoulder_yaw_link: geometry collision mesh filename=meshes/right_shoulder_yaw_link.stl; visual mesh filename=meshes/right_shoulder_yaw_link.stl
- link right_wrist_pitch_link: geometry collision mesh filename=meshes/right_wrist_pitch_link.stl; visual mesh filename=meshes/right_wrist_pitch_link.stl
- link right_wrist_roll_link: geometry collision mesh filename=meshes/right_wrist_roll_link.stl; visual mesh filename=meshes/right_wrist_roll_link.stl
- link right_wrist_yaw_link: geometry collision mesh filename=meshes/right_wrist_yaw_link.stl; visual mesh filename=meshes/right_wrist_yaw_link.stl
- link torso_link: geometry collision mesh filename=meshes/torso_link.stl; visual mesh filename=meshes/torso_link.stl
- link waist_roll_link: geometry visual mesh filename=meshes/waist_roll_link.stl
- link waist_support_link: geometry collision mesh filename=meshes/waist_support_link.stl; visual mesh filename=meshes/waist_support_link.stl
- link waist_yaw_link: geometry visual mesh filename=meshes/waist_yaw_link.stl
